Commit message: Update module category

File: UsageTemplate/Resources/URDF/Demo_5/Demo_5.urdf (robot description, URDF)
Before this commit: robot Demo_5_Robot, 16 links, 15 joints
Links:
- link unit_1: geometry visual mesh filename=meshes/SpiRob_unit_1.stl
- link unit_10: geometry visual mesh filename=meshes/SpiRob_unit_10.stl
- link unit_11: geometry visual mesh filename=meshes/SpiRob_unit_11.stl
- link unit_12: geometry visual mesh filename=meshes/SpiRob_unit_12.stl
- link unit_13: geometry visual mesh filename=meshes/SpiRob_unit_13.stl
- link unit_14: geometry visual mesh filename=meshes/SpiRob_unit_14.stl
- link unit_15: geometry visual mesh filename=meshes/SpiRob_unit_15.stl
- link unit_16: geometry visual mesh filename=meshes/SpiRob_unit_16.stl
- link unit_2: geometry visual mesh filename=meshes/SpiRob_unit_2.stl
- link unit_3: geometry visual mesh filename=meshes/SpiRob_unit_3.stl
- link unit_4: geometry visual mesh filename=meshes/SpiRob_unit_4.stl
- link unit_5: geometry visual mesh filename=meshes/SpiRob_unit_5.stl
- link unit_6: geometry visual mesh filename=meshes/SpiRob_unit_6.stl
- link unit_7: geometry visual mesh filename=meshes/SpiRob_unit_7.stl
- link unit_8: geometry visual mesh filename=meshes/SpiRob_unit_8.stl
- link unit_9: geometry visual mesh filename=meshes/SpiRob_unit_9.stl
